File: PCB/FPGC5IOboard/FPGC4IOboard.sch (KiCad schematic (older format))
At the start: 174 parts, among them J1 Conn_PS2_Mini_Din_6, J10 Conn_GPIO_Ext, J11 Conn_SPI_Ext, J12 Conn_Headphone_Jack, J13 Conn_W5500_1, J14 Conn_W5500_2, J2 Conn_NES, J4 Conn_NConfig, J6 Conn_Stacked_USB, J7 Conn_Debug_U8, J8 Conn_Debug_U7, J9 Conn_UART_Ext, Q1 BSS138, Q2 BSS138, Q3 BC847, Q4 BC847, SW1 SW_Push_Rst, SW2 SW_Slide, SW3 SW_Push_Config, U2 CH376T, U3 CH376T, U4 Conn_02x32_U7, U5 Conn_02x32_U8, U7 W25Q128JVS, U8 ESP32-WROOM-32U, U9 UDA1334ATS, Y1 12MHz, Y2 12MHz

Commit message: Fixed vertical position of NTSC output. Restored GPIO pin assignments and moved NTSC to the extra pins on the bottom of the PCB. Worked a tiny bit on the new PCB version. Added a cython base version of the Ccompiler, since moving to C++ will litterally take forever and maybe cython will be fast enough when some static typing is done
Parts:
- removed J2: Conn_NES, SNES:SNES_controller_port, symbol FPGC4IOboard-rescue:Conn_01x07-Connector_Generic
- added D?: LED, symbol Device:LED
- added J?: Conn_RCA_Audio, RCJ013:CUI_RCJ-013, symbol Connector:Conn_Coaxial
- added R?: 1k, Resistor_SMD:R_0805_2012Metric_Pad1.15x1.40mm_HandSolder, symbol FPGC4IOboard-rescue:R-Device
- added R?: 10k, Resistor_SMD:R_0805_2012Metric_Pad1.15x1.40mm_HandSolder, symbol FPGC4IOboard-rescue:R-Device
- F?: value 500mA -> 0.75A
- J?: value Conn_RCA -> Conn_RCA_Video
- SW?: footprint switch:switchAngled -> (none)
Connections:
- net +3V3: now also R?.2
- net CRT_AUDIO: now also J?.1 (In), R?.1; no longer C38.1, J12.2 (Pin_2), R49.1
- net GND: now also J?.2 (Ext)
- new net: D?.2 (A), R?.1
- new net LED_VideoOutput: D?.1 (K)
- new net Tip: C38.1, J12.2 (Pin_2), R49.1, R?.2
- no-connect marks 65 -> 63
Other:
- note added: "8bit DAC (NTSC Video)"
- note added: "Can move to the back now, since good USB keyboard support"
- note added: "If too many leds, use some kind of multiplexing"
- note added: "TODO: add tvs diodes"
- note added: "TODO: better physical switch"
- note added: "TODO: look into adding 5v somewhere (like other development boards do)"
- note added: "TODO: look into easy to solder SMD connector \nlike the breakout board"
- note removed: "8bit DAC"
- note removed: "NES controller port"
- moved on the sheet: J?, R?
Changed lines of the file:
@@
 $EndDescr
 $Comp
-L FPGC4IOboard-rescue:Conn_01x07-Connector_Generic J2
-U 1 1 5E2A11F1
-P 1300 3950
-F 0 "J2" H 1350 3450 50  0000 L CNN
-F 1 "Conn_NES" H 1150 3550 50  0000 L CNN
-F 2 "SNES:SNES_controller_port" H 1300 3950 50  0001 C CNN
-F 3 "~" H 1300 3950 50  0001 C CNN
-	1    1300 3950
-	-1   0    0    1
-$EndComp
-$Comp
-L FPGC4IOboard-rescue:GND-power #PWR014
-U 1 1 5E2AF5E8
-P 1650 3700
-F 0 "#PWR014" H 1650 3450 50  0001 C CNN
-F 1 "GND" H 1750 3600 50  0000 C CNN
-F 2 "" H 1650 3700 50  0001 C CNN
-F 3 "" H 1650 3700 50  0001 C CNN
-	1    1650 3700
-	1    0    0    -1
-$EndComp
-Wire Wire Line
-	1650 3650 1500 3650
-$Comp
-L FPGC4IOboard-rescue:+3.3V-power #PWR015
-U 1 1 5E2B1790
-P 1700 4350
-F 0 "#PWR015" H 1700 4200 50  0001 C CNN
-F 1 "+3.3V" H 1850 4400 50  0000 C CNN
-F 2 "" H 1700 4350 50  0001 C CNN
-F 3 "" H 1700 4350 50  0001 C CNN
-	1    1700 4350
-	1    0    0    -1
-$EndComp
-NoConn ~ 1500 3750
-NoConn ~ 1500 3850
-$Comp
 L FPGC4IOboard-rescue:GND-power #PWR0108
 U 1 1 5E3B478B
@@
 Text Notes 14400 750  0    50   ~ 0
 IO Headers
-Wire Wire Line
-	1550 4250 1500 4250
-Text Notes 2100 3450 2    50   ~ 0
-NES controller port
 $Comp
 L FPGC4IOboard-rescue:Conn_01x04-Connector_Generic J12
@@
 Text Label 17550 1350 1    50   ~ 0
 IO_GP
-Text GLabel 1650 4150 2    50   Input ~ 0
-NES_CLK
-Text GLabel 1650 4050 2    50   Input ~ 0
-NES_Latch
-Text GLabel 1650 3950 2    50   Output ~ 0
-NES_Data
-Wire Wire Line
-	1500 4150 1650 4150
-Wire Wire Line
-	1500 4050 1650 4050
-Wire Wire Line
-	1500 3950 1650 3950
 Text GLabel 4700 1100 2    50   Input ~ 0
 PS2_CLK
@@
 	13200 9400 22850 9400
 Wire Wire Line
-	1650 3650 1650 3700
-Wire Wire Line
-	1550 4250 1550 4350
-Wire Wire Line
-	1550 4350 1700 4350
-Wire Notes Line
-	950  3350 2150 3350
-Wire Notes Line
-	2150 3350 2150 4750
-Wire Notes Line
-	2150 4750 950  4750
-Wire Notes Line
-	950  3350 950  4750
-Wire Wire Line
 	18100 3400 18050 3400
 Wire Wire Line
@@
 Wire Wire Line
 	9250 7000 9250 7050
-Text GLabel 17100 14100 2    50   Output ~ 0
+Text GLabel 17650 13850 2    50   Output ~ 0
 CRT_AUDIO
 Wire Wire Line
 	17050 14250 17050 14100
-Wire Wire Line
-	17050 14100 17100 14100
 Connection ~ 17050 14250
 Text GLabel 9850 9700 1    50   Input ~ 0
@@
 P 19850 7000
 F 0 "F?" V 19650 6950 50  0000 L CNN
-F 1 "500mA" V 19750 6900 50  0000 L CNN
+F 1 "0.75A" V 19750 6900 50  0000 L CNN
 F 2 "Fuse:Fuse_1812_4532Metric_Pad1.30x3.40mm_HandSolder" V 19780 7000 50  0001 C CNN
 F 3 "~" H 19850 7000 50  0001 C CNN
@@
 F 0 "SW?" V 20000 6300 50  0000 L CNN
 F 1 "SW_Power" V 20100 6100 50  0000 L CNN
-F 2 "switch:switchAngled" H 20150 6600 50  0001 C CNN
+F 2 "" H 20150 6600 50  0001 C CNN
 F 3 "~" H 20150 6600 50  0001 C CNN
 	1    20150 6600
@@
 L FPGC4IOboard-rescue:R-Device R?
 U 1 1 666D70BF
-P 10700 13200
-F 0 "R?" V 10600 13100 50  0000 C CNN
-F 1 "75" V 10600 13300 50  0000 C CNN
-F 2 "Resistor_SMD:R_0805_2012Metric_Pad1.15x1.40mm_HandSolder" V 10630 13200 50  0001 C CNN
-F 3 "~" H 10700 13200 50  0001 C CNN
-	1    10700 13200
+P 10850 13200
+F 0 "R?" V 10750 13100 50  0000 C CNN
+F 1 "75" V 10750 13300 50  0000 C CNN
+F 2 "Resistor_SMD:R_0805_2012Metric_Pad1.15x1.40mm_HandSolder" V 10780 13200 50  0001 C CNN
+F 3 "~" H 10850 13200 50  0001 C CNN
+	1    10850 13200
 	0    -1   -1   0
 $EndComp
@@
 Wire Wire Line
 	10350 12600 10350 13200
-Wire Wire Line
-	10550 13200 10350 13200
-Connection ~ 10350 13200
 $Comp
 L FPGC4IOboard-rescue:C-Device C?
@@
 L Connector:Conn_Coaxial J?
 U 1 1 685B9D15
-P 11150 13200
-F 0 "J?" H 11250 13175 50  0000 L CNN
-F 1 "Conn_RCA" H 11250 13084 50  0000 L CNN
-F 2 "RCJ013:CUI_RCJ-013" H 11150 13200 50  0001 C CNN
-F 3 " ~" H 11150 13200 50  0001 C CNN
-	1    11150 13200
+P 11300 13200
+F 0 "J?" H 11400 13175 50  0000 L CNN
+F 1 "Conn_RCA_Video" H 11000 13350 50  0000 L CNN
+F 2 "RCJ013:CUI_RCJ-013" H 11300 13200 50  0001 C CNN
+F 3 " ~" H 11300 13200 50  0001 C CNN
+	1    11300 13200
 	1    0    0    -1
 $EndComp
 Wire Wire Line
-	10950 13200 10850 13200
+	11100 13200 11000 13200
 $Comp
 L FPGC4IOboard-rescue:GND-power #PWR?
@@
 L FPGC4IOboard-rescue:GND-power #PWR?
 U 1 1 686B50E5
-P 11150 13500
-F 0 "#PWR?" H 11150 13250 50  0001 C CNN
-F 1 "GND" H 11000 13450 50  0000 C CNN
-F 2 "" H 11150 13500 50  0001 C CNN
-F 3 "" H 11150 13500 50  0001 C CNN
-	1    11150 13500
+P 11300 13500
+F 0 "#PWR?" H 11300 13250 50  0001 C CNN
+F 1 "GND" H 11150 13450 50  0000 C CNN
+F 2 "" H 11300 13500 50  0001 C CNN
+F 3 "" H 11300 13500 50  0001 C CNN
+	1    11300 13500
 	1    0    0    -1
 $EndComp
 Wire Wire Line
-	11150 13400 11150 13500
+	11300 13400 11300 13500
 Wire Notes Line
 	5950 12050 11650 12050
@@
 	5950 14200 5950 12050
 Text Notes 6000 12150 0    50   ~ 0
-8bit DAC
+8bit DAC (NTSC Video)
 Text GLabel 1150 7000 3    50   Input ~ 0
 LED_Booted
@@
 Connection ~ 2050 8600
 NoConn ~ 2250 10000
+$Comp
+L Connector:Conn_Coaxial J?
+U 1 1 617BE518
+P 11300 12350
+F 0 "J?" H 11400 12325 50  0000 L CNN
+F 1 "Conn_RCA_Audio" H 11000 12500 50  0000 L CNN
+F 2 "RCJ013:CUI_RCJ-013" H 11300 12350 50  0001 C CNN
+F 3 " ~" H 11300 12350 50  0001 C CNN
+	1    11300 12350
+	1    0    0    -1
+$EndComp
+Wire Wire Line
+	11100 12350 11000 12350
+$Comp
+L FPGC4IOboard-rescue:GND-power #PWR?
+U 1 1 617BE51F
+P 11300 12650
+F 0 "#PWR?" H 11300 12400 50  0001 C CNN
+F 1 "GND" H 11150 12600 50  0000 C CNN
+F 2 "" H 11300 12650 50  0001 C CNN
+F 3 "" H 11300 12650 50  0001 C CNN
+	1    11300 12650
+	1    0    0    -1
+$EndComp
+Wire Wire Line
+	11300 12550 11300 12650
+Text Notes 1200 8500 0    50   ~ 0
+TODO: look into easy to solder SMD connector \nlike the breakout board
+$Comp
+L FPGC4IOboard-rescue:R-Device R?
+U 1 1 618862D9
+P 5000 6350
+F 0 "R?" H 4850 6250 50  0000 C CNN
+F 1 "1k" H 4850 6350 50  0000 C CNN
+F 2 "Resistor_SMD:R_0805_2012Metric_Pad1.15x1.40mm_HandSolder" V 4930 6350 50  0001 C CNN
+F 3 "~" H 5000 6350 50  0001 C CNN
+	1    5000 6350
+	1    0    0    1
+$EndComp
+Text GLabel 5000 7000 3    50   Input ~ 0
+LED_VideoOutput
+$Comp
+L Device:LED D?
+U 1 1 618862E0
+P 5000 6750
+F 0 "D?" V 4947 6830 50  0000 L CNN
+F 1 "LED" V 5038 6830 50  0000 L CNN
+F 2 "" H 5000 6750 50  0001 C CNN
+F 3 "~" H 5000 6750 50  0001 C CNN
+	1    5000 6750
+	0    -1   -1   0
+$EndComp
+Wire Wire Line
+	5000 6500 5000 6600
+Wire Wire Line
+	5000 6900 5000 7000
+$Comp
+L FPGC4IOboard-rescue:+3.3V-power #PWR?
+U 1 1 618862E8
+P 5000 6100
+F 0 "#PWR?" H 5000 5950 50  0001 C CNN
+F 1 "+3.3V" H 4850 6200 50  0000 C CNN
+F 2 "" H 5000 6100 50  0001 C CNN
+F 3 "" H 5000 6100 50  0001 C CNN
+	1    5000 6100
+	1    0    0    -1
+$EndComp
+Wire Wire Line
+	5000 6100 5000 6200
+Text Notes 1200 7650 0    50   ~ 0
+If too many leds, use some kind of multiplexing
+Text Notes 2300 750  0    50   ~ 0
+Can move to the back now, since good USB keyboard support
+Text Notes 14500 2200 0    50   ~ 0
+TODO: look into adding 5v somewhere (like other development boards do)
+Text Notes 20300 6650 0    50   ~ 0
+TODO: better physical switch
+Text GLabel 11000 12350 0    50   Input ~ 0
+CRT_AUDIO
+Wire Wire Line
+	10350 13200 10700 13200
+Connection ~ 10350 13200
+$Comp
+L FPGC4IOboard-rescue:R-Device R?
+U 1 1 61AA0A74
+P 17400 13850
+F 0 "R?" V 17300 13750 50  0000 C CNN
+F 1 "10k" V 17300 13950 50  0000 C CNN
+F 2 "Resistor_SMD:R_0805_2012Metric_Pad1.15x1.40mm_HandSolder" V 17330 13850 50  0001 C CNN
+F 3 "~" H 17400 13850 50  0001 C CNN
+	1    17400 13850
+	0    1    1    0
+$EndComp
+Wire Wire Line
+	17550 13850 17650 13850
+Wire Wire Line
+	17250 13850 17200 13850
+Wire Wire Line
+	17200 13850 17200 14100
+Wire Wire Line
+	17050 14100 17200 14100
+Text Notes 2500 10600 0    50   ~ 0
+TODO: add tvs diodes
 $EndSCHEMATC

Commit message: Added many connectors and stuffs to new PCB
Parts:
- added U? (x2): SRV05-4, Package_TO_SOT_SMD:SOT-23-6, symbol RCJ-013:SRV05-4
- J?: value HDMI_A -> HDMI_conn; footprint (none) -> RCJ013:HDMI_connector_19
- J?: footprint Connector_USB:USB_Micro-B_Wuerth_629105150521 -> RCJ013:MicroUSB_G30
Connections:
- net +5V: now also U?.5, U?.5
- net GND: now also U?.2, U?.2
- net HDMI_D2+: now reaches J?.1 (D2+)
- net HDMI_D2+: now also U?.4
- net HDMI_CLK+: now reaches J?.10 (CK+)
- net HDMI_CLK+: now also U?.1
- net HDMI_CLK-: now reaches J?.12 (CK-)
- net HDMI_CLK-: now also U?.6
- net HDMI_D2-: now reaches J?.3 (D2-)
- net HDMI_D2-: now also U?.3
- net HDMI_D1+: now reaches J?.4 (D1+)
- net HDMI_D1+: now also U?.6
- net HDMI_D1-: now reaches J?.6 (D1-)
- net HDMI_D1-: now also U?.1
- net HDMI_D0+: now reaches J?.7 (D0+)
- net HDMI_D0+: now also U?.3
- net HDMI_D0-: now reaches J?.9 (D0-)
- net HDMI_D0-: now also U?.4
- net NES_CLK: no longer names the net of U4.11 (Pin_11)
- net NES_Data: no longer names the net of U4.15 (Pin_15)
- net NES_Latch: no longer names the net of U4.13 (Pin_13)
- no-connect marks 63 -> 74
Other:
- note added: "HDMI OUT"
- note added: "TODO: look into an alternative for audio"
- note removed: "If too many leds, use some kind of multiplexing"
- note removed: "TODO: add tvs diodes"
- note removed: "TODO: look into easy to solder SMD connector \nlike the breakout board"
Changed lines of the file:
@@
 Text GLabel 12050 6650 3    50   Output ~ 0
 FPGC4_DTR
-Text GLabel 9750 6650 3    50   Input ~ 0
-NES_CLK
-Text GLabel 9850 6650 3    50   Input ~ 0
-NES_Latch
-Text GLabel 9950 6650 3    50   Output ~ 0
-NES_Data
-Text GLabel 9550 6650 3    50   Input ~ 0
-PS2_CLK
 Text GLabel 9650 6650 3    50   BiDi ~ 0
 PS2_Data
@@
 F 0 "J?" H 21520 11047 50  0000 R CNN
 F 1 "USB_B_Micro" H 21520 11138 50  0000 R CNN
-F 2 "Connector_USB:USB_Micro-B_Wuerth_629105150521" H 21900 11100 50  0001 C CNN
+F 2 "RCJ013:MicroUSB_G30" H 21900 11100 50  0001 C CNN
 F 3 "~" H 21900 11100 50  0001 C CNN
 	1    21750 11150
@@
 Wire Wire Line
 	9200 12800 9200 12900
-Text GLabel 11550 9250 1    50   Input ~ 0
+Text GLabel 11900 8950 1    50   Output ~ 0
 DAC_D6
-Text GLabel 11450 9250 1    50   Input ~ 0
+Text GLabel 11800 8950 1    50   Output ~ 0
 DAC_D5
-Text GLabel 11350 9250 1    50   Input ~ 0
+Text GLabel 11700 8950 1    50   Output ~ 0
 DAC_D4
-Text GLabel 11250 9250 1    50   Input ~ 0
+Text GLabel 11600 8950 1    50   Output ~ 0
 DAC_D3
-Text GLabel 11150 9250 1    50   Input ~ 0
+Text GLabel 11500 8950 1    50   Output ~ 0
 DAC_D2
-Text GLabel 11050 9250 1    50   Input ~ 0
+Text GLabel 11400 8950 1    50   Output ~ 0
 DAC_D1
-Text GLabel 10950 9250 1    50   Input ~ 0
+Text GLabel 11300 8950 1    50   Output ~ 0
 DAC_D0
-Text GLabel 11650 9250 1    50   Input ~ 0
+Text GLabel 12000 8950 1    50   Output ~ 0
 DAC_D7
 $Comp
@@
 U 1 1 61E88954
 P 1850 10100
-F 0 "J?" H 2280 10054 50  0000 L CNN
-F 1 "HDMI_A" H 2280 10145 50  0000 L CNN
-F 2 "" H 1875 10100 50  0001 C CNN
+F 0 "J?" H 1400 9200 50  0000 L CNN
+F 1 "HDMI_conn" H 1100 9100 50  0000 L CNN
+F 2 "RCJ013:HDMI_connector_19" H 1875 10100 50  0001 C CNN
 F 3 "https://en.wikipedia.org/wiki/HDMI" H 1875 10100 50  0001 C CNN
 	1    1850 10100
@@
 Wire Wire Line
 	11300 12550 11300 12650
-Text Notes 1200 8500 0    50   ~ 0
-TODO: look into easy to solder SMD connector \nlike the breakout board
 $Comp
 L FPGC4IOboard-rescue:R-Device R?
@@
 Wire Wire Line
 	5000 6100 5000 6200
-Text Notes 1200 7650 0    50   ~ 0
-If too many leds, use some kind of multiplexing
 Text Notes 2300 750  0    50   ~ 0
 Can move to the back now, since good USB keyboard support
@@
 Wire Wire Line
 	17050 14100 17200 14100
-Text Notes 2500 10600 0    50   ~ 0
-TODO: add tvs diodes
+Text GLabel 9550 6650 3    50   Input ~ 0
+PS2_CLK
+Text Notes 13450 9750 0    50   ~ 0
+TODO: look into an alternative for audio
+NoConn ~ 18150 5450
+NoConn ~ 18150 5650
+NoConn ~ 18150 5750
+NoConn ~ 18150 5850
+NoConn ~ 18150 5950
+NoConn ~ 19300 10850
+NoConn ~ 19300 10950
+NoConn ~ 19300 11050
+NoConn ~ 19300 11150
+NoConn ~ 20100 11350
+NoConn ~ 18950 6150
+$Comp
+L RCJ-013:SRV05-4 U?
+U 1 1 625E169B
+P 3100 9550
+F 0 "U?" H 3075 9965 50  0000 C CNN
+F 1 "SRV05-4" H 3075 9874 50  0000 C CNN
+F 2 "Package_TO_SOT_SMD:SOT-23-6" H 3200 9200 50  0001 C CNN
+F 3 "https://katalog.we-online.de/pbs/datasheet/82400102.pdf" H 3100 9300 50  0001 C CNN
+	1    3100 9550
+	1    0    0    -1
+$EndComp
+$Comp
+L RCJ-013:SRV05-4 U?
+U 1 1 625E4C72
+P 3100 11600
+F 0 "U?" H 3075 12015 50  0000 C CNN
+F 1 "SRV05-4" H 3075 11924 50  0000 C CNN
+F 2 "Package_TO_SOT_SMD:SOT-23-6" H 3200 11250 50  0001 C CNN
+F 3 "https://katalog.we-online.de/pbs/datasheet/82400102.pdf" H 3100 11350 50  0001 C CNN
+	1    3100 11600
+	1    0    0    -1
+$EndComp
+Wire Wire Line
+	2250 10300 2550 10300
+Wire Wire Line
+	2250 10400 3450 10400
+Wire Wire Line
+	2250 10500 2700 10500
+Wire Wire Line
+	2250 10600 2700 10600
+Wire Wire Line
+	2250 10700 3450 10700
+Wire Wire Line
+	2250 10800 2550 10800
+Wire Wire Line
+	2250 10900 3550 10900
+Wire Wire Line
+	2250 10200 3550 10200
+Wire Wire Line
+	3350 9400 3550 9400
+Wire Wire Line
+	3550 9400 3550 10200
+Connection ~ 3550 10200
+Wire Wire Line
+	3550 10200 4200 10200
+Wire Wire Line
+	2800 9400 2550 9400
+Wire Wire Line
+	2550 9400 2550 10300
+Connection ~ 2550 10300
+Wire Wire Line
+	2550 10300 4200 10300
+Wire Wire Line
+	2800 9700 2700 9700
+Wire Wire Line
+	2700 9700 2700 10500
+Connection ~ 2700 10500
+Wire Wire Line
+	2700 10500 4200 10500
+Wire Wire Line
+	3350 9700 3450 9700
+Wire Wire Line
+	3450 9700 3450 10400
+Connection ~ 3450 10400
+Wire Wire Line
+	3450 10400 4200 10400
+$Comp
+L FPGC4IOboard-rescue:GND-power #PWR?
+U 1 1 630B0A32
+P 2700 9550
+F 0 "#PWR?" H 2700 9300 50  0001 C CNN
+F 1 "GND" H 2700 9600 50  0000 C CNN
+F 2 "" H 2700 9550 50  0001 C CNN
+F 3 "" H 2700 9550 50  0001 C CNN
+	1    2700 9550
+	1    0    0    -1
+$EndComp
+Wire Wire Line
+	2800 9550 2700 9550
+$Comp
+L FPGC4IOboard-rescue:+5V-power #PWR?
+U 1 1 631524B2
+P 3450 9550
+F 0 "#PWR?" H 3450 9400 50  0001 C CNN
+F 1 "+5V" H 3450 9500 50  0000 C CNN
+F 2 "" H 3450 9550 50  0001 C CNN
+F 3 "" H 3450 9550 50  0001 C CNN
+	1    3450 9550
+	1    0    0    -1
+$EndComp
+Wire Wire Line
+	3350 9550 3450 9550
+$Comp
+L FPGC4IOboard-rescue:GND-power #PWR?
+U 1 1 631F5ACB
+P 2700 11600
+F 0 "#PWR?" H 2700 11350 50  0001 C CNN
+F 1 "GND" H 2700 11650 50  0000 C CNN
+F 2 "" H 2700 11600 50  0001 C CNN
+F 3 "" H 2700 11600 50  0001 C CNN
+	1    2700 11600
+	1    0    0    -1
+$EndComp
+Wire Wire Line
+	2800 11600 2700 11600
+$Comp
+L FPGC4IOboard-rescue:+5V-power #PWR?
+U 1 1 632994F8
+P 3450 11600
+F 0 "#PWR?" H 3450 11450 50  0001 C CNN
+F 1 "+5V" H 3450 11550 50  0000 C CNN
+F 2 "" H 3450 11600 50  0001 C CNN
+F 3 "" H 3450 11600 50  0001 C CNN
+	1    3450 11600
+	1    0    0    -1
+$EndComp
+Wire Wire Line
+	3350 11600 3450 11600
+Wire Wire Line
+	2550 10800 2550 11750
+Wire Wire Line
+	2550 11750 2800 11750
+Connection ~ 2550 10800
+Wire Wire Line
+	2550 10800 4200 10800
+Wire Wire Line
+	3350 11750 3550 11750
+Wire Wire Line
+	3550 11750 3550 10900
+Connection ~ 3550 10900
+Wire Wire Line
+	3550 10900 4200 10900
+Wire Wire Line
+	3450 10700 3450 11450
+Wire Wire Line
+	3450 11450 3350 11450
+Connection ~ 3450 10700
+Wire Wire Line
+	3450 10700 4200 10700
+Wire Wire Line
+	2700 10600 2700 11450
+Wire Wire Line
+	2700 11450 2800 11450
+Connection ~ 2700 10600
+Wire Wire Line
+	2700 10600 4200 10600
+Text GLabel 10350 8950 1    50   Output ~ 0
+HDMI_CLK-
+Text GLabel 10450 8950 1    50   Output ~ 0
+HDMI_CLK+
+Text GLabel 10550 8950 1    50   Output ~ 0
+HDMI_D0-
+Text GLabel 10650 8950 1    50   Output ~ 0
+HDMI_D0+
+Text GLabel 10750 8950 1    50   Output ~ 0
+HDMI_D1-
+Text GLabel 10850 8950 1    50   Output ~ 0
+HDMI_D1+
+Text GLabel 10950 8950 1    50   Output ~ 0
+HDMI_D2-
+Text GLabel 11050 8950 1    50   Output ~ 0
+HDMI_D2+
+Wire Notes Line
+	1350 8450 4750 8450
+Wire Notes Line
+	4750 8450 4750 11950
+Wire Notes Line
+	4750 11950 1350 11950
+Wire Notes Line
+	1350 11950 1350 8450
+Text Notes 4350 8550 0    50   ~ 0
+HDMI OUT
+Text GLabel 4200 10200 2    50   Input ~ 0
+HDMI_CLK-
+Text GLabel 4200 10300 2    50   Input ~ 0
+HDMI_CLK+
+Text GLabel 4200 10400 2    50   Input ~ 0
+HDMI_D0-
+Text GLabel 4200 10500 2    50   Input ~ 0
+HDMI_D0+
+Text GLabel 4200 10600 2    50   Input ~ 0
+HDMI_D1-
+Text GLabel 4200 10700 2    50   Input ~ 0
+HDMI_D1+
+Text GLabel 4200 10800 2    50   Input ~ 0
+HDMI_D2-
+Text GLabel 4200 10900 2    50   Input ~ 0
+HDMI_D2+
 $EndSCHEMATC
