File: PCB/FPGC5IOboard/FPGC4IOboard.sch (KiCad schematic (older format))
At the start: 138 parts, among them IC1 CS4344-CZZ, J1 Conn_PS2_Mini_Din_6, J10 Conn_GPIO_Ext, J11 Conn_SPI_Ext, J12 Conn_Headphone_Jack, J13 Conn_W5500_1, J14 Conn_W5500_2, J15 USB_B_Micro, J2 HDMI_conn, J3 Conn_RCA_Audio, J4 Conn_NConfig, J5 Conn_RCA_Video, J6 Conn_Stacked_USB, J9 Conn_UART_Ext, Q1 BSS138, Q2 BSS138, SW1 SW_Push_Rst, SW2 SW_Slide, SW3 SW_Push_Config, SW4 SW_Power, U1 SRV05-4, U2 CH376T, U3 CH376T, U4 Conn_02x32_U7, U5 Conn_02x32_U8, U6 SRV05-4, U7 W25Q128JVS, U8 ADA4841-1YRJ, U9 CH340G, Y1 12MHz, Y2 12MHz, Y3 12MHz

Commit message: Basically finished the new PCB design
Parts:
- added C10, C11, C33, C34, C35: 47uF, Capacitor_SMD:C_0805_2012Metric_Pad1.18x1.45mm_HandSolder, symbol FPGC4IOboard-rescue:C-Device
- renumbered IC1 to U10
Connections:
- net +3V3: now also C10.2, C11.1
- net +5V: now also C33.2, C34.1, C35.1
- net GND: now also C10.1, C11.2, C33.1, C34.2, C35.2
Changed lines of the file:
@@
 Connection ~ 9350 7050
 Wire Wire Line
-	9250 6150 9250 5750
-Wire Wire Line
 	9250 5750 9350 5750
 Wire Wire Line
@@
 Connection ~ 9350 5750
 Wire Wire Line
-	9350 6050 9350 6150
-Wire Wire Line
 	9350 6650 9350 6700
 Wire Wire Line
@@
 	0    -1   -1   0
 $EndComp
-$Comp
-L FPGC4IOboard-rescue:C-Device C17
-U 1 1 7518F417
-P 10800 4200
-F 0 "C17" V 10650 4050 50  0000 L CNN
-F 1 "100nF" V 10650 4250 50  0000 L CNN
-F 2 "Capacitor_SMD:C_0805_2012Metric_Pad1.18x1.45mm_HandSolder" H 10838 4050 50  0001 C CNN
-F 3 "~" H 10800 4200 50  0001 C CNN
-	1    10800 4200
-	0    1    -1   0
-$EndComp
-$Comp
-L FPGC4IOboard-rescue:GND-power #PWR055
-U 1 1 7534C6FB
-P 11100 4100
-F 0 "#PWR055" H 11100 3850 50  0001 C CNN
-F 1 "GND" H 11150 3950 50  0000 C CNN
-F 2 "" H 11100 4100 50  0001 C CNN
-F 3 "" H 11100 4100 50  0001 C CNN
-	1    11100 4100
-	1    0    0    -1
-$EndComp
 Wire Wire Line
 	10950 3950 11000 3950
 Wire Wire Line
 	10950 4200 11000 4200
-Wire Wire Line
-	11000 4200 11000 4050
-Wire Wire Line
-	11000 4050 11100 4050
-Connection ~ 11000 4050
-Wire Wire Line
-	11000 4050 11000 3950
-Wire Wire Line
-	11100 4050 11100 4100
 $Comp
 L FPGC4IOboard-rescue:R-Device R26
@@
 $EndComp
 Wire Wire Line
-	9250 10200 9250 10600
+	9250 10200 9250 10550
 Wire Wire Line
 	9450 10200 9450 10600
 Wire Wire Line
-	9350 10200 9350 10300
+	9350 10200 9350 10250
 $Comp
 L FPGC4IOboard-rescue:+5V-power #PWR083
@@
 U 1 1 61627EF4
 P 20300 7150
-F 0 "C32" H 20100 7100 50  0000 L CNN
+F 0 "C32" H 20050 7100 50  0000 L CNN
 F 1 "220uF" H 19950 7200 50  0000 L CNN
 F 2 "Capacitor_THT:CP_Radial_D5.0mm_P2.00mm" H 20338 7000 50  0001 C CNN
@@
 	16550 12000 16700 12000
 $Comp
-L CS4344-CZZ:CS4344-CZZ IC1
+L CS4344-CZZ:CS4344-CZZ U10
 U 1 1 61BB5EA1
 P 16750 11250
-F 0 "IC1" H 17450 11515 50  0000 C CNN
+F 0 "U10" H 17450 11515 50  0000 C CNN
 F 1 "CS4344-CZZ" H 17450 11424 50  0000 C CNN
 F 2 "RCJ013:SOP50P490X110-10N" H 18000 11350 50  0001 L CNN
@@
 NoConn ~ 10850 10200
 NoConn ~ 10950 10200
+$Comp
+L FPGC4IOboard-rescue:C-Device C11
+U 1 1 618A876B
+P 9100 10400
+F 0 "C11" H 9250 10450 50  0000 L CNN
+F 1 "47uF" H 9250 10350 50  0000 L CNN
+F 2 "Capacitor_SMD:C_0805_2012Metric_Pad1.18x1.45mm_HandSolder" H 9138 10250 50  0001 C CNN
+F 3 "~" H 9100 10400 50  0001 C CNN
+	1    9100 10400
+	-1   0    0    -1
+$EndComp
+Wire Wire Line
+	9100 10550 9250 10550
+Connection ~ 9250 10550
+Wire Wire Line
+	9250 10550 9250 10600
+Wire Wire Line
+	9100 10250 9350 10250
+Connection ~ 9350 10250
+Wire Wire Line
+	9350 10250 9350 10300
+$Comp
+L FPGC4IOboard-rescue:C-Device C10
+U 1 1 619DE131
+P 9100 5950
+F 0 "C10" H 9250 6000 50  0000 L CNN
+F 1 "47uF" H 9250 5900 50  0000 L CNN
+F 2 "Capacitor_SMD:C_0805_2012Metric_Pad1.18x1.45mm_HandSolder" H 9138 5800 50  0001 C CNN
+F 3 "~" H 9100 5950 50  0001 C CNN
+	1    9100 5950
+	-1   0    0    -1
+$EndComp
+Wire Wire Line
+	9250 5750 9250 5800
+Wire Wire Line
+	9100 5800 9250 5800
+Connection ~ 9250 5800
+Wire Wire Line
+	9250 5800 9250 6150
+Wire Wire Line
+	9100 6100 9350 6100
+Wire Wire Line
+	9350 6050 9350 6100
+Connection ~ 9350 6100
+Wire Wire Line
+	9350 6100 9350 6150
+$Comp
+L FPGC4IOboard-rescue:C-Device C33
+U 1 1 61E23DE4
+P 20550 6950
+F 0 "C33" V 20700 6900 50  0000 L CNN
+F 1 "47uF" V 20800 6850 50  0000 L CNN
+F 2 "Capacitor_SMD:C_0805_2012Metric_Pad1.18x1.45mm_HandSolder" H 20588 6800 50  0001 C CNN
+F 3 "~" H 20550 6950 50  0001 C CNN
+	1    20550 6950
+	0    1    -1   0
+$EndComp
+Wire Wire Line
+	20300 6950 20400 6950
+$Comp
+L FPGC4IOboard-rescue:GND-power #PWR04
+U 1 1 61E96521
+P 20750 7000
+F 0 "#PWR04" H 20750 6750 50  0001 C CNN
+F 1 "GND" H 20750 6850 50  0000 C CNN
+F 2 "" H 20750 7000 50  0001 C CNN
+F 3 "" H 20750 7000 50  0001 C CNN
+	1    20750 7000
+	-1   0    0    -1
+$EndComp
+Wire Wire Line
+	20700 6950 20750 6950
+Wire Wire Line
+	20750 6950 20750 7000
+Wire Wire Line
+	10600 4200 10600 4450
+Wire Wire Line
+	10600 4450 10650 4450
+Connection ~ 10600 4200
+Wire Wire Line
+	10600 4450 10600 4650
+Wire Wire Line
+	10600 4650 10650 4650
+Connection ~ 10600 4450
+Wire Wire Line
+	11000 4200 11000 4450
+Wire Wire Line
+	11000 4450 10950 4450
+Connection ~ 11000 4200
+Wire Wire Line
+	11000 4650 10950 4650
+Connection ~ 11000 4450
+Wire Wire Line
+	11000 4550 11100 4550
+Wire Wire Line
+	11100 4550 11100 4600
+Wire Wire Line
+	11000 4450 11000 4550
+Wire Wire Line
+	11000 4550 11000 4650
+Connection ~ 11000 4550
+Wire Wire Line
+	11000 3950 11000 4200
+$Comp
+L FPGC4IOboard-rescue:GND-power #PWR055
+U 1 1 7534C6FB
+P 11100 4600
+F 0 "#PWR055" H 11100 4350 50  0001 C CNN
+F 1 "GND" H 11200 4500 50  0000 C CNN
+F 2 "" H 11100 4600 50  0001 C CNN
+F 3 "" H 11100 4600 50  0001 C CNN
+	1    11100 4600
+	1    0    0    -1
+$EndComp
+$Comp
+L FPGC4IOboard-rescue:C-Device C34
+U 1 1 61F79B4B
+P 10800 4450
+F 0 "C34" V 10750 4300 50  0000 L CNN
+F 1 "47uF" V 10800 4000 50  0000 L CNN
+F 2 "Capacitor_SMD:C_0805_2012Metric_Pad1.18x1.45mm_HandSolder" H 10838 4300 50  0001 C CNN
+F 3 "~" H 10800 4450 50  0001 C CNN
+	1    10800 4450
+	0    -1   1    0
+$EndComp
+$Comp
+L FPGC4IOboard-rescue:C-Device C17
+U 1 1 7518F417
+P 10800 4200
+F 0 "C17" V 10850 4250 50  0000 L CNN
+F 1 "100nF" V 10800 4450 50  0000 L CNN
+F 2 "Capacitor_SMD:C_0805_2012Metric_Pad1.18x1.45mm_HandSolder" H 10838 4050 50  0001 C CNN
+F 3 "~" H 10800 4200 50  0001 C CNN
+	1    10800 4200
+	0    1    -1   0
+$EndComp
+$Comp
+L FPGC4IOboard-rescue:C-Device C35
+U 1 1 61F7E9CB
+P 10800 4650
+F 0 "C35" V 10850 4750 50  0000 L CNN
+F 1 "47uF" V 10850 4400 50  0000 L CNN
+F 2 "Capacitor_SMD:C_0805_2012Metric_Pad1.18x1.45mm_HandSolder" H 10838 4500 50  0001 C CNN
+F 3 "~" H 10800 4650 50  0001 C CNN
+	1    10800 4650
+	0    -1   1    0
+$EndComp
 $EndSCHEMATC
