File: PCB/FPGC5IOboard/FPGC4IOboard.kicad_pcb (KiCad board)
At the start: 4 copper layers, 105.4 x 137.7 mm, 170 parts, among them J1 Conn_PS2_Mini_Din_6, J10 Conn_GPIO_Ext, J11 Conn_SPI_Ext, J12 Conn_Headphone_Jack, J13 Conn_W5500_1, J14 Conn_W5500_2, J15 USB_B_Mini, J16 USB_B_Mini, J2 Conn_SNES, J3 Conn_RGBs, J4 Conn_NConfig, J5 Conn_VGA, J6 Conn_Stacked_USB, J7 Conn_Debug_U8, J8 Conn_Debug_U7, J9 Conn_UART_Ext, Q1 BSS138, Q2 BSS138, Q3 BC847, Q4 BC847, SW1 SW_Push_Rst, SW2 SW_Slide, SW3 SW_Push_Config, SW4 SW_Power, U1 ADV7123, U10 FT232RL, U11 FT232RL, U2 CH376T, U3 CH376T, U4 Conn_02x32_U7, U5 Conn_02x32_U8, U6 ADV7123, U7 W25Q128JVS, U8 ESP32-WROOM-32U, U9 UDA1334ATS, Y1 12MHz, Y2 12MHz

Commit message: Started on PCB layouting
Parts:
- removed C33: 47uF, Capacitor_THT:CP_Radial_D4.0mm_P2.00mm
- removed C34: 10uF, Capacitor_SMD:C_0805_2012Metric_Pad1.15x1.40mm_HandSolder
- removed C35: 1uF, Capacitor_SMD:C_0805_2012Metric_Pad1.15x1.40mm_HandSolder
- removed C36, C40, C42, C43, C44, C46, C47, C49: 100nF, Capacitor_SMD:C_0805_2012Metric_Pad1.15x1.40mm_HandSolder
- removed C37, C41, C45: 22uF, Capacitor_SMD:C_0805_2012Metric_Pad1.15x1.40mm_HandSolder
- removed C38, C39: 10nF, Capacitor_SMD:C_0805_2012Metric_Pad1.15x1.40mm_HandSolder
- removed C48: 220uF, Capacitor_THT:CP_Radial_D5.0mm_P2.00mm
- removed J16: USB_B_Mini, Connector_USB:USB_Mini-B_Lumberg_2486_01_Horizontal
- removed LOGO: , logo:LOGO
- removed Q3, Q4: BC847, Package_TO_SOT_SMD:SOT-23
- removed R62, R65: 10k, Resistor_SMD:R_0805_2012Metric_Pad1.15x1.40mm_HandSolder
- removed R63, R64: 1k, Resistor_SMD:R_0805_2012Metric_Pad1.15x1.40mm_HandSolder
- removed R66, R67, R68, R69: 0, Resistor_SMD:R_0805_2012Metric_Pad1.15x1.40mm_HandSolder
- removed the REF** at (109.2, 88.9)
- removed the REF** at (109.2, 94.0)
- removed the REF** at (109.2, 99.1)
- removed the REF** at (166.4, 25.4)
- removed the REF** at (68.6, 155.4)
- removed the REF** at (166.4, 155.4)
- removed the REF** at (68.6, 25.4)
- removed U10, U11: FT232RL, SmallSMD:SSOP-28_5.3x10.2mm_P0.65mm
- added C28: 22pF, Capacitor_SMD:C_0805_2012Metric_Pad1.18x1.45mm_HandSolder, F.Cu at (318.9, 92.0)
- added C4: 3.3uF, Capacitor_SMD:C_0805_2012Metric_Pad1.18x1.45mm_HandSolder, F.Cu at (318.9, 98.0)
- added D10: LED, LED_SMD:LED_0805_2012Metric_Pad1.15x1.40mm_HandSolder, F.Cu at (81.0, 97.2)
- added D11: Green_LED, LED_SMD:LED_0805_2012Metric_Pad1.15x1.40mm_HandSolder, F.Cu at (81.0, 76.8)
- added D12: Red_LED, LED_SMD:LED_0805_2012Metric_Pad1.15x1.40mm_HandSolder, F.Cu at (81.0, 74.3)
- added D5: LED, LED_SMD:LED_0805_2012Metric_Pad1.15x1.40mm_HandSolder, F.Cu at (81.0, 81.9)
- added D6: LED, LED_SMD:LED_0805_2012Metric_Pad1.15x1.40mm_HandSolder, F.Cu at (81.0, 99.7)
- added D7: LED, LED_SMD:LED_0805_2012Metric_Pad1.15x1.40mm_HandSolder, F.Cu at (81.0, 92.1)
- added D8: LED, LED_SMD:LED_0805_2012Metric_Pad1.15x1.40mm_HandSolder, F.Cu at (81.0, 87.0)
- added D9: LED, LED_SMD:LED_0805_2012Metric_Pad1.15x1.40mm_HandSolder, F.Cu at (81.0, 94.6)
- added IC1: CS4344-CZZ, RCJ013:SOP50P490X110-10N, F.Cu at (259.1, 115.1)
- added REF**: MountingHole_3.2mm_M3_Pad, MountingHole:MountingHole_3.2mm_M3_Pad, F.Cu at (166.4, 37.5)
- added REF**: MountingHole_3.2mm_M3_Pad, MountingHole:MountingHole_3.2mm_M3_Pad, F.Cu at (82.5, 37.5)
- added REF**: MountingHole_3.2mm_M3_Pad, MountingHole:MountingHole_3.2mm_M3_Pad, F.Cu at (82.5, 132.7)
- added REF**: MountingHole_3.2mm_M3_Pad, MountingHole:MountingHole_3.2mm_M3_Pad, F.Cu at (166.4, 132.7)
- added Y3: 12MHz, Crystal:Crystal_HC49-4H_Vertical, F.Cu at (134.6, 85.1)
- C1, C31: footprint Capacitor_SMD:C_0805_2012Metric_Pad1.15x1.40mm_HandSolder -> Capacitor_SMD:C_0805_2012Metric_Pad1.18x1.45mm_HandSolder; moved to F.Cu
- C11, C12, C13, C14, C15, C17, C18, C19, C2, C20, C21, C25, C5, C8, C9: footprint Capacitor_SMD:C_0805_2012Metric_Pad1.15x1.40mm_HandSolder -> Capacitor_SMD:C_0805_2012Metric_Pad1.18x1.45mm_HandSolder
- C22: value 100nF -> 1uF; footprint Capacitor_SMD:C_0805_2012Metric_Pad1.15x1.40mm_HandSolder -> Capacitor_SMD:C_0805_2012Metric_Pad1.18x1.45mm_HandSolder
- C23: value 100nF -> 3.3uF; footprint Capacitor_SMD:C_0805_2012Metric_Pad1.15x1.40mm_HandSolder -> Capacitor_SMD:C_0805_2012Metric_Pad1.18x1.45mm_HandSolder
- C26: value 100nF -> 3.3uF; footprint Capacitor_SMD:C_0805_2012Metric_Pad1.15x1.40mm_HandSolder -> Capacitor_SMD:C_0805_2012Metric_Pad1.18x1.45mm_HandSolder; moved to F.Cu
- C27: value 10uF -> 22pF; footprint Capacitor_SMD:C_0805_2012Metric_Pad1.15x1.40mm_HandSolder -> Capacitor_SMD:C_0805_2012Metric_Pad1.18x1.45mm_HandSolder; moved to F.Cu
- C29: value 10uF -> 2.7nF; footprint Capacitor_SMD:C_0805_2012Metric_Pad1.15x1.40mm_HandSolder -> Capacitor_SMD:C_0805_2012Metric_Pad1.18x1.45mm_HandSolder; moved to F.Cu
- C3: value 100nF -> 100pf; footprint Capacitor_SMD:C_0805_2012Metric_Pad1.15x1.40mm_HandSolder -> Capacitor_SMD:C_0805_2012Metric_Pad1.18x1.45mm_HandSolder
- C30: value 100nF -> 2.7nF; footprint Capacitor_SMD:C_0805_2012Metric_Pad1.15x1.40mm_HandSolder -> Capacitor_SMD:C_0805_2012Metric_Pad1.18x1.45mm_HandSolder; moved to F.Cu
- C32: value 47uF -> 220uF; footprint Capacitor_THT:CP_Radial_D4.0mm_P2.00mm -> Capacitor_THT:CP_Radial_D5.0mm_P2.00mm
- C6: value 100nF -> 10uF; footprint Capacitor_SMD:C_0805_2012Metric_Pad1.15x1.40mm_HandSolder -> Capacitor_SMD:C_0805_2012Metric_Pad1.18x1.45mm_HandSolder
- D1, D3: value Green_LED -> LED
- D2, D4: value Red_LED -> LED
- F1: value 500mA -> 0.75A; footprint Fuse:Fuse_1812_4532Metric_Pad1.30x3.40mm_HandSolder -> RCJ013:Fuse_1812
- J1: footprint Custom:Connector_Mini-DIN_Female_6Pin_2rows -> RCJ013:PS2
- J12: footprint Custom:TRRS-PJ-320A -> RCJ013:TRRS-PJ-320A
- J15: value USB_B_Mini -> USB_B_Micro; footprint Connector_USB:USB_Mini-B_Lumberg_2486_01_Horizontal -> RCJ013:MicroUSB_G30
- J2: value Conn_SNES -> HDMI_conn; footprint SNES:SNES_controller_port -> RCJ013:HDMI_connector_19
- J3: value Conn_RGBs -> Conn_RCA_Audio; footprint Custom:DSUB9_CRT -> RCJ013:CUI_RCJ-013
- J5: value Conn_VGA -> Conn_RCA_Video; footprint Custom:VGA_EDAC -> RCJ013:CUI_RCJ-013-Min
- Q1, Q2, Y1, Y2: moved to F.Cu
- R1, R2, R29, R30: value 75 -> 1k; footprint Resistor_SMD:R_0805_2012Metric_Pad1.15x1.40mm_HandSolder -> Resistor_SMD:R_0805_2012Metric_Pad1.20x1.40mm_HandSolder; moved to F.Cu
- R10, R11, R4, R5, R60, R61: footprint Resistor_SMD:R_0805_2012Metric_Pad1.15x1.40mm_HandSolder -> Resistor_SMD:R_0805_2012Metric_Pad1.20x1.40mm_HandSolder; moved to F.Cu
- R12: value 33 -> 1k; footprint Resistor_SMD:R_0805_2012Metric_Pad1.15x1.40mm_HandSolder -> Resistor_SMD:R_0805_2012Metric_Pad1.20x1.40mm_HandSolder
- R13, R32: value 510 -> 1k; footprint Resistor_SMD:R_0805_2012Metric_Pad1.15x1.40mm_HandSolder -> Resistor_SMD:R_0805_2012Metric_Pad1.20x1.40mm_HandSolder
- R14: value 4.7k -> 2k; footprint Resistor_SMD:R_0805_2012Metric_Pad1.15x1.40mm_HandSolder -> Resistor_SMD:R_0805_2012Metric_Pad1.20x1.40mm_HandSolder
- R15, R17, R18, R19, R21, R23, R24, R25, R26, R27, R33, R35, R36, R54, R55, R56, R57, R6, R7, R70, R71, R72, R73, R8: footprint Resistor_SMD:R_0805_2012Metric_Pad1.15x1.40mm_HandSolder -> Resistor_SMD:R_0805_2012Metric_Pad1.20x1.40mm_HandSolder
- R16, R20, R22: value 100 -> 1k; footprint Resistor_SMD:R_0805_2012Metric_Pad1.15x1.40mm_HandSolder -> Resistor_SMD:R_0805_2012Metric_Pad1.20x1.40mm_HandSolder
- R28, R3: value 75 -> 2k; footprint Resistor_SMD:R_0805_2012Metric_Pad1.15x1.40mm_HandSolder -> Resistor_SMD:R_0805_2012Metric_Pad1.20x1.40mm_HandSolder; moved to F.Cu
- R31: value 33 -> 2k; footprint Resistor_SMD:R_0805_2012Metric_Pad1.15x1.40mm_HandSolder -> Resistor_SMD:R_0805_2012Metric_Pad1.20x1.40mm_HandSolder
- R34: value 4.7k -> 1k; footprint Resistor_SMD:R_0805_2012Metric_Pad1.15x1.40mm_HandSolder -> Resistor_SMD:R_0805_2012Metric_Pad1.20x1.40mm_HandSolder
- R37, R40, R46: value 10k -> 2k; footprint Resistor_SMD:R_0805_2012Metric_Pad1.15x1.40mm_HandSolder -> Resistor_SMD:R_0805_2012Metric_Pad1.20x1.40mm_HandSolder; moved to F.Cu
- R38, R39, R41, R42: value 10k -> 1k; footprint Resistor_SMD:R_0805_2012Metric_Pad1.15x1.40mm_HandSolder -> Resistor_SMD:R_0805_2012Metric_Pad1.20x1.40mm_HandSolder; moved to F.Cu
- R43: value 0 -> 2k; footprint Resistor_SMD:R_0805_2012Metric_Pad1.15x1.40mm_HandSolder -> Resistor_SMD:R_0805_2012Metric_Pad1.20x1.40mm_HandSolder; moved to F.Cu
- R44, R45: value 0 -> 1k; footprint Resistor_SMD:R_0805_2012Metric_Pad1.15x1.40mm_HandSolder -> Resistor_SMD:R_0805_2012Metric_Pad1.20x1.40mm_HandSolder; moved to F.Cu
- R47: value 220k -> 1.6k; footprint Resistor_SMD:R_0805_2012Metric_Pad1.15x1.40mm_HandSolder -> Resistor_SMD:R_0805_2012Metric_Pad1.20x1.40mm_HandSolder; moved to F.Cu
- R48: value 220k -> 100; footprint Resistor_SMD:R_0805_2012Metric_Pad1.15x1.40mm_HandSolder -> Resistor_SMD:R_0805_2012Metric_Pad1.20x1.40mm_HandSolder; moved to F.Cu
- R49: value 100 -> 75; footprint Resistor_SMD:R_0805_2012Metric_Pad1.15x1.40mm_HandSolder -> Resistor_SMD:R_0805_2012Metric_Pad1.20x1.40mm_HandSolder; moved to F.Cu
- R50: value 100 -> 0; footprint Resistor_SMD:R_0805_2012Metric_Pad1.15x1.40mm_HandSolder -> Resistor_SMD:R_0805_2012Metric_Pad1.20x1.40mm_HandSolder; moved to F.Cu
- R51: value 1k -> 0; footprint Resistor_SMD:R_0805_2012Metric_Pad1.15x1.40mm_HandSolder -> Resistor_SMD:R_0805_2012Metric_Pad1.20x1.40mm_HandSolder
- R52, R53: value 1k -> 10k; footprint Resistor_SMD:R_0805_2012Metric_Pad1.15x1.40mm_HandSolder -> Resistor_SMD:R_0805_2012Metric_Pad1.20x1.40mm_HandSolder
- R58, R59: value 10k -> 470; footprint Resistor_SMD:R_0805_2012Metric_Pad1.15x1.40mm_HandSolder -> Resistor_SMD:R_0805_2012Metric_Pad1.20x1.40mm_HandSolder; moved to F.Cu
- R9: value 330 -> 2k; footprint Resistor_SMD:R_0805_2012Metric_Pad1.15x1.40mm_HandSolder -> Resistor_SMD:R_0805_2012Metric_Pad1.20x1.40mm_HandSolder; moved to F.Cu
- SW4: footprint switch:switchAngled -> RCJ013:SS12D06
- U1, U6: value ADV7123 -> SRV05-4; footprint Package_QFP:LQFP-48_7x7mm_P0.5mm -> Package_TO_SOT_SMD:SOT-23-6
- U2, U3: footprint SmallSMD:SSOP-20_5.3x7.2mm_P0.65mm -> RCJ013:SSOP-20_5.3x7.2mm_P0.65mm
- U7: footprint Package_SO:SOIC-8_5.23x5.23mm_P1.27mm -> RCJ013:SOIC-8_5.23x5.23mm_P1.27mm
- U8: value ESP32-WROOM-32U -> ADA4841-1YRJ; footprint RF_Module:ESP32-WROOM-32U -> Package_TO_SOT_SMD:SOT-23-6; moved to F.Cu
- U9: value UDA1334ATS -> CH340G; footprint Package_SO:SSOP-16_4.4x5.2mm_P0.65mm -> Package_SO:SOIC-16_3.9x9.9mm_P1.27mm; moved to F.Cu
- moved R51 285.1 mm to (355.2, 76.1), turned to 0 degrees
- moved R5 282.7 mm to (351.3, 70.1), turned to 0 degrees
- moved R10 282.5 mm to (356.1, 66.4), turned to 0 degrees
- moved R23 272.3 mm to (348.4, 90.9), turned to 0 degrees
- moved R6 268.2 mm to (345.6, 79.1), turned to 0 degrees
- moved Q2 268.0 mm to (331.0, 110.4), turned to 0 degrees
- moved R52 266.1 mm to (338.9, 93.5), turned to 0 degrees
- moved R18 265.5 mm to (335.9, 87.6), turned to 0 degrees
- moved R3 265.3 mm to (356.1, 69.4), turned to 0 degrees
- moved C1 264.7 mm to (335.3, 78.6)
- moved J7 260.3 mm to (338.5, 39.4), turned to 270 degrees
- moved R26 259.6 mm to (355.0, 85.0), turned to 0 degrees
- moved R70 259.1 mm to (350.4, 79.1), turned to 0 degrees
- moved R21 256.5 mm to (331.2, 106.7), turned to 0 degrees
- moved C24 256.4 mm to (340.3, 68.2), turned to 0 degrees
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Connections:
- net VUSB renamed Net-(J15-Pad1)
- C18 pad 1: +3V3 -> GND
- C18 pad 2: Net-(C18-Pad2) -> +3V3
- C19 pad 2: Net-(C19-Pad2) -> GND
- C2 pad 1: +3V3 -> +5V
- C2 pad 2: Net-(C2-Pad2) -> GND
- C22 pad 1: GND -> +3V3
- C22 pad 2: +3V3 -> GND
- C23 pad 1: +3V3 -> Net-(C23-Pad1)
- C23 pad 2: GND -> Net-(C23-Pad2)
- C26 pad 2: GND -> Net-(C26-Pad2)
- C27 pad 1: Net-(C26-Pad1) -> Net-(C27-Pad1)
- C29 pad 1: Net-(C29-Pad1) -> GND
- C29 pad 2: GND -> Net-(C29-Pad2)
- C3 pad 1: +3V3 -> Net-(C3-Pad1)
- C30 pad 1: Net-(C29-Pad1) -> Net-(C30-Pad1)
- C31 pad 1: Net-(C31-Pad1) -> GND
- C31 pad 2: GND -> Net-(C31-Pad2)
- C32 pad 1: Net-(C32-Pad1) -> Net-(C31-Pad2)
- C32 pad 2: Net-(C32-Pad2) -> GND
- C5 pad 1: GND -> Net-(C4-Pad1)
- C5 pad 2: +3V3 -> GND
- C6 pad 1: +3V3 -> Net-(C6-Pad1)
- D1 pad 1: Net-(D1-Pad1) -> LED_Booted
- D2 pad 1: Net-(D2-Pad1) -> LED_Eth
- D3 pad 1: Net-(D3-Pad1) -> LED_Flash
- D4 pad 1: Net-(D4-Pad1) -> LED_USB0
- F1 pad 1: Net-(C46-Pad2) -> Net-(C31-Pad2)
- J1 pad 7: (no net) -> GND
- J12 pad 2: CRT_AUDIO -> Audio_Mono
- J15 pad 2: /USB_FPGC4_D1- -> /USB_FPGC_D1-
- J15 pad 3: /USB_FPGC4_D1+ -> /USB_FPGC_D1+
- J2 pad 1: +3V3 -> HDMI_D2+
- J2 pad 2: SNES_CLK -> GND
- J2 pad 3: SNES_Latch -> HDMI_D2-
- J2 pad 4: SNES_Data -> HDMI_D1+
- J2 pad 5: Net-(J2-Pad5) -> GND
- J2 pad 6: Net-(J2-Pad6) -> HDMI_D1-
- J2 pad 7: GND -> HDMI_D0+
- J3 pad 1: Net-(J3-Pad1) -> Audio_Mono
- J3 pad 2: /RGBS_SYNC -> GND
- J5 pad 1: /VGA_R -> Net-(J5-Pad1)
- J5 pad 2: /VGA_G -> GND
- R1 pad 1: GND -> Net-(D1-Pad2)
- R1 pad 2: /RGBS_BLUE -> +3V3
- R12 pad 1: CRT_CLK -> Net-(D3-Pad2)
- R12 pad 2: Net-(R12-Pad2) -> +3V3
- R13 pad 2: GND -> Net-(R13-Pad2)
- R14 pad 1: +3V3 -> DAC_D1
- R14 pad 2: Net-(R14-Pad2) -> Net-(R13-Pad2)
- R16 pad 1: +3V3 -> Net-(D4-Pad2)
- R16 pad 2: Net-(J3-Pad1) -> +3V3
- R2 pad 1: GND -> Net-(D2-Pad2)
- R2 pad 2: /RGBS_GREEN -> +3V3
- R20 pad 1: /VGA_VS -> Net-(R13-Pad2)
- R20 pad 2: VGA_VSYNC -> Net-(R20-Pad2)
- R22 pad 1: /VGA_HS -> Net-(D5-Pad2)
- R22 pad 2: VGA_HSYNC -> +3V3
- R28 pad 1: GND -> DAC_D2
- R28 pad 2: /VGA_B -> Net-(R20-Pad2)
- R29 pad 1: GND -> Net-(R20-Pad2)
- R29 pad 2: /VGA_G -> Net-(R29-Pad2)
- R3 pad 1: GND -> DAC_D0
- R3 pad 2: /RGBS_RED -> Net-(R13-Pad1)
- R30 pad 1: GND -> Net-(D6-Pad2)
- R30 pad 2: /VGA_R -> +3V3
- R31 pad 1: VGA_CLK -> DAC_D3
- R31 pad 2: Net-(R31-Pad2) -> Net-(R29-Pad2)
- R32 pad 1: Net-(R32-Pad1) -> Net-(R29-Pad2)
- R32 pad 2: GND -> Net-(R32-Pad2)
- R34 pad 1: +3V3 -> Net-(D7-Pad2)
- R34 pad 2: Net-(R34-Pad2) -> +3V3
- R37 pad 1: Net-(R37-Pad1) -> DAC_D4
- R37 pad 2: GND -> Net-(R32-Pad2)
- R38 pad 1: Net-(R38-Pad1) -> Net-(R32-Pad2)
- R38 pad 2: GND -> Net-(R38-Pad2)
- R39 pad 1: Net-(R39-Pad1) -> Net-(D8-Pad2)
- R39 pad 2: GND -> +3V3
- R40 pad 1: Net-(R40-Pad1) -> DAC_D5
- R40 pad 2: GND -> Net-(R38-Pad2)
- R41 pad 1: Net-(R41-Pad1) -> Net-(D9-Pad2)
- R41 pad 2: GND -> +3V3
- R42 pad 1: Net-(R42-Pad1) -> Net-(R38-Pad2)
- R42 pad 2: GND -> Net-(R42-Pad2)
- R43 pad 1: Net-(R43-Pad1) -> DAC_D6
- R43 pad 2: Net-(R43-Pad2) -> Net-(R42-Pad2)
- R44 pad 1: +3V3 -> Net-(D10-Pad2)
- R44 pad 2: Net-(C26-Pad1) -> +3V3
- R45 pad 1: Net-(C29-Pad1) -> Net-(R42-Pad2)
- R45 pad 2: +3V3 -> Net-(R45-Pad2)
- R46 pad 1: Net-(C35-Pad1) -> DAC_D7
- R46 pad 2: +3V3 -> Net-(R45-Pad2)
- R47 pad 1: GND -> Net-(R45-Pad2)
- R47 pad 2: Net-(C32-Pad2) -> GND
- R48 pad 1: Net-(C33-Pad2) -> Net-(C3-Pad2)
- R48 pad 2: GND -> Net-(C3-Pad1)
- R49 pad 1: CRT_AUDIO -> Net-(C3-Pad1)
- R49 pad 2: Net-(C32-Pad2) -> Net-(J5-Pad1)
- R50 pad 1: /Ring1 -> FPGC_TX
- R50 pad 2: Net-(C33-Pad2) -> Net-(D11-Pad1)
- R51 pad 1: Net-(C43-Pad2) -> Net-(D12-Pad1)
- R51 pad 2: Net-(D1-Pad2) -> FPGC_RX
- R52 pad 1: Net-(C43-Pad2) -> Net-(D11-Pad2)
- R52 pad 2: Net-(D2-Pad2) -> +3V3
- R53 pad 1: Net-(R53-Pad1) -> +3V3
- R53 pad 2: FPGC4_DTR -> Net-(D12-Pad2)
- R54 pad 1: FPGC4_TX -> /USB_FPGC_D2-
- R54 pad 2: Net-(R54-Pad2) -> /USB_FPGC_D1-
- R55 pad 1: Net-(R55-Pad1) -> /USB_FPGC_D2+
- R55 pad 2: FPGC4_RX -> /USB_FPGC_D1+
- R56 pad 1: Net-(R54-Pad2) -> GND
- R56 pad 2: +3V3 -> Net-(C23-Pad2)
- R57 pad 1: +3V3 -> Net-(C26-Pad2)
- R57 pad 2: Net-(R55-Pad1) -> GND
- R58 pad 1: Net-(Q3-Pad1) -> Net-(C29-Pad2)
- R58 pad 2: Net-(Q4-Pad2) -> Net-(C23-Pad2)
- R59 pad 1: Net-(Q4-Pad1) -> Net-(C30-Pad1)
- R59 pad 2: Net-(Q3-Pad2) -> Net-(C26-Pad2)
- R60 pad 1: Net-(R60-Pad1) -> Audio_Mono
- R60 pad 2: Net-(R60-Pad2) -> Net-(C29-Pad2)
- R61 pad 1: Net-(R61-Pad1) -> /Ring1
- R61 pad 2: Net-(R61-Pad2) -> Net-(C30-Pad1)
- R9 pad 1: /RGBS_SYNC -> Net-(R13-Pad1)
- R9 pad 2: CRT_CSYNC -> GND
- SW1 pad : (no net) -> GND
- SW3 pad : (no net) -> GND
- SW4 pad : (no net) -> GND
- SW4 pad 2: Net-(C46-Pad2) -> Net-(C31-Pad2)
- U1 pad 1: GND -> HDMI_CLK+
- U1 pad 3: GND -> HDMI_D0+
- U1 pad 4: GND -> HDMI_D0-
- U1 pad 5: GND -> +5V
- U1 pad 6: GND -> HDMI_CLK-
- U4 pad 11: SNES_CLK -> LED_Booted
- U4 pad 13: SNES_Latch -> LED_Eth
- U4 pad 15: SNES_Data -> LED_Flash
- U4 pad 17: Net-(U4-Pad17) -> LED_USB0
- U4 pad 19: ESP32_RX2 -> LED_USB1
- U4 pad 21: ESP32_TX2 -> Net-(U4-Pad21)
- U4 pad 55: FPGC4_RX -> FPGC_RX
- U4 pad 57: FPGC4_DTR -> FPGC_DTR
- U4 pad 59: FPGC4_TX -> FPGC_TX
- U5 pad 18: Net-(J7-Pad1) -> LED_I2S
- U5 pad 19: CRT_CSYNC -> DAC_D7
- U5 pad 20: Net-(J7-Pad3) -> LED_FSX
- U5 pad 21: CRT_CLK -> DAC_D6
- U5 pad 22: Net-(J7-Pad5) -> LED_SPImode
- U5 pad 23: CRT_B0 -> DAC_D5
- U5 pad 24: Net-(J7-Pad7) -> LED_VideoOutput
- U5 pad 25: CRT_B1 -> DAC_D4
- U5 pad 26: Net-(J7-Pad9) -> LED_PS2
- U5 pad 27: CRT_G0 -> DAC_D3
- U5 pad 28: Net-(J7-Pad11) -> I2S_MCLK
- U5 pad 29: CRT_G1 -> DAC_D2
- U5 pad 30: Net-(J7-Pad13) -> I2S_LRCLK
- U5 pad 31: CRT_G2 -> DAC_D1
- U5 pad 32: Net-(J7-Pad15) -> I2S_SCLK
- U5 pad 33: CRT_R0 -> DAC_D0
- U5 pad 34: Net-(J7-Pad17) -> I2S_SDIN
- U5 pad 35: CRT_R1 -> Net-(U5-Pad35)
- U5 pad 36: Net-(J7-Pad19) -> Net-(J7-Pad1)
- U5 pad 37: CRT_R2 -> Net-(U5-Pad37)
- U5 pad 38: Net-(U5-Pad38) -> Net-(J7-Pad3)
- U5 pad 39: VGA_HSYNC -> Net-(U5-Pad39)
- U5 pad 40: Net-(U5-Pad40) -> Net-(J7-Pad5)
- U5 pad 41: VGA_VSYNC -> Net-(U5-Pad41)
- U5 pad 42: Net-(U5-Pad42) -> Net-(J7-Pad7)
- U5 pad 43: VGA_CLK -> Net-(U5-Pad43)
- U5 pad 44: Net-(U5-Pad44) -> Net-(J7-Pad9)
- U5 pad 45: VGA_B0 -> HDMI_CLK-
- U5 pad 46: Net-(U5-Pad46) -> Net-(J7-Pad11)
- U5 pad 47: VGA_B1 -> HDMI_CLK+
- U5 pad 48: Net-(U5-Pad48) -> Net-(J7-Pad13)
- U5 pad 49: VGA_G0 -> HDMI_D0-
- U5 pad 50: Net-(U5-Pad50) -> Net-(J7-Pad15)
- U5 pad 51: VGA_G1 -> HDMI_D0+
- U5 pad 52: Net-(U5-Pad52) -> Net-(J7-Pad17)
- U5 pad 53: VGA_G2 -> HDMI_D1-
- U5 pad 54: Net-(U5-Pad54) -> Net-(J7-Pad19)
- U5 pad 55: VGA_R0 -> HDMI_D1+
- U5 pad 57: VGA_R1 -> HDMI_D2-
- U5 pad 59: VGA_R2 -> HDMI_D2+
- U6 pad 1: GND -> HDMI_D1-
- U6 pad 3: GND -> HDMI_D2-
- U6 pad 4: GND -> HDMI_D2+
- U6 pad 5: GND -> +5V
- U6 pad 6: GND -> HDMI_D1+
- U8 pad 1: GND -> Net-(C3-Pad1)
- U8 pad 2: +3V3 -> GND
- U8 pad 3: Net-(C35-Pad1) -> Net-(R45-Pad2)
- U8 pad 4: Net-(U8-Pad4) -> Net-(C3-Pad2)
- U8 pad 5: Net-(U8-Pad5) -> +5V
- U8 pad 6: Net-(U8-Pad6) -> +5V
- U9 pad 1: Net-(U8-Pad11) -> GND
- U9 pad 10: Net-(R40-Pad1) -> Net-(U9-Pad10)
- U9 pad 11: Net-(R42-Pad1) -> Net-(U9-Pad11)
- U9 pad 12: Net-(C31-Pad1) -> Net-(U9-Pad12)
- U9 pad 13: Net-(C29-Pad1) -> FPGC_DTR
- U9 pad 14: Net-(C32-Pad1) -> Net-(U9-Pad14)
- U9 pad 15: GND -> Net-(U9-Pad15)
- U9 pad 16: Net-(C33-Pad1) -> +3V3
- U9 pad 2: Net-(R43-Pad1) -> Net-(D12-Pad1)
- U9 pad 3: Net-(U8-Pad8) -> Net-(D11-Pad1)
- U9 pad 4: Net-(C26-Pad1) -> +3V3
- U9 pad 5: GND -> /USB_FPGC_D2+
- U9 pad 6: Net-(R37-Pad1) -> /USB_FPGC_D2-
- U9 pad 7: Net-(R39-Pad1) -> Net-(C28-Pad2)
- U9 pad 8: Net-(R38-Pad1) -> Net-(C27-Pad1)
- U9 pad 9: Net-(R41-Pad1) -> Net-(U9-Pad9)
Routing:
- net +5V: track 314.6 -> 0.00 mm, vias 4 -> 0
- net GND: track 258.6 -> 0.00 mm, vias 85 -> 0
- net Net-(J4-Pad1): track 141.4 -> 0.00 mm, vias 5 -> 0
- net Net-(D4-Pad1): track 132.7 -> 0.00 mm, vias 3 -> 0
- net Net-(D2-Pad1): track 132.3 -> 0.00 mm, vias 2 -> 0
- net Net-(D3-Pad1): track 126.6 -> 0.00 mm, vias 3 -> 0
- net Net-(D1-Pad1): track 126.6 -> 0.00 mm, vias 2 -> 0
- net +3V3: track 122.4 -> 0.00 mm, vias 37 -> 0
- net Net-(C43-Pad2): track 120.9 -> 0.00 mm, vias 2 -> 0
- net CRT_AUDIO: track 120.8 -> 0.00 mm, vias 1 -> 0
- net Net-(C49-Pad2): track 113.0 -> 0.00 mm, vias 3 -> 0
- net Net-(J8-Pad1): track 59.2 -> 0.00 mm
- net Net-(J8-Pad3): track 58.6 -> 0.00 mm
- net Net-(J8-Pad5): track 57.5 -> 0.00 mm
- net Net-(J8-Pad7): track 57.1 -> 0.00 mm
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Other:
- board size 105.4 x 137.7 mm -> 91.4 x 102.9 mm
- board text added: "Audio"
- board text added: "ETH"
- board text added: "Flash"
- board text added: "GPU"
- board text added: "HDMI"
- board text added: "K21"
- board text added: "LOGO"
- board text added: "Power"
- board text added: "SPI Mode"
- board text added: "U7"
- board text added: "U8"
- board text added: "USB0"
- board text added: "USB1"
- board text removed: "APU"
- board text removed: "Audio Out"
- board text removed: "CONN_U7"
- board text removed: "CONN_U8"
- board text removed: "ESP32 USB"
- board text removed: "FPGC4"
- board text removed: "FPGC4 I/O Board"
- board text removed: "OFF"
- board text removed: "ON"
- board text removed: "Power/Data"
- board text removed: "RGBS"
- board text removed: "Reboot"
- board text removed: "Reset"
- board text removed: "SNES"
- board text removed: "SPI Flash"
- board text removed: "USB"
- board text removed: "V2.0"
- board text removed: "VGA"
- board text removed: "W5500"
- board text removed: "nConfig"

Commit message: PCB v3 initial routing done. Need to optimize and finish silkscreen layer
Parts:
- removed C10: 100uF, Capacitor_THT:CP_Radial_D4.0mm_P2.00mm
- removed C11: 100nF, Capacitor_SMD:C_0805_2012Metric_Pad1.18x1.45mm_HandSolder
- removed J7: Conn_Debug_U8, Connector_PinHeader_2.54mm:PinHeader_2x10_P2.54mm_Vertical
- removed J8: Conn_Debug_U7, Connector_PinHeader_2.54mm:PinHeader_2x10_P2.54mm_Vertical
- removed R24, R27: 0, Resistor_SMD:R_0805_2012Metric_Pad1.20x1.40mm_HandSolder
- added LOGO: , RCJ013:LOGO, F.Cu at (100.3, 50.2)
- C1, C17, C31, Q1, Q2, R1, R10, R11, R12, R15, R16, R17, R2, R21, R22, R23, R25, R26, R30, R34, R35, R36, R39, R4, R41, R44, R5, R52, R53, R6, R7, R8, Y1, Y2, Y3: moved to B.Cu
- C24, C7: value 100uF -> 47uF; footprint Capacitor_THT:CP_Radial_D4.0mm_P2.00mm -> Capacitor_SMD:C_0805_2012Metric_Pad1.18x1.45mm_HandSolder; moved to B.Cu
- J3: footprint RCJ013:CUI_RCJ-013 -> RCJ013:CUI_RCJ-013-Min
- R18: value 10K -> 0R; moved to B.Cu
- moved R44 266.1 mm to (85.5, 97.2)
- moved R53 265.0 mm to (85.5, 74.3), turned to 180 degrees
- moved R6 262.4 mm to (84.7, 51.4), turned to 180 degrees
- moved R23 262.2 mm to (89.2, 51.2), turned to 90 degrees
- moved R16 258.4 mm to (85.5, 79.4)
- moved R12 258.3 mm to (85.5, 84.5)
- moved R70 257.6 mm to (93.0, 69.8)
- moved C24 257.0 mm to (90.2, 127.0)
- moved R39 255.4 mm to (85.5, 87.0)
- moved R15 254.7 mm to (84.7, 46.4), turned to 180 degrees
- moved R18 254.6 mm to (83.8, 123.5), turned to 270 degrees
- moved R52 253.9 mm to (85.5, 76.8)
- moved R8 252.8 mm to (84.7, 48.9), turned to 180 degrees
- moved R17 250.5 mm to (84.7, 43.8), turned to 180 degrees
- moved R34 248.6 mm to (85.5, 92.1)
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Connections:
- C16 pad 1: /+5V1 -> +5V
- C17 pad 2: /+5V1 -> +5V
- C24 pad 1: +3V3 -> GND
- C24 pad 2: GND -> +3V3
- C31 pad 2: Net-(C31-Pad2) -> +5V
- C32 pad 1: Net-(C31-Pad2) -> +5V
- F1 pad 1: Net-(C31-Pad2) -> Net-(F1-Pad1)
- F1 pad 2: +5V -> Net-(F1-Pad2)
- J15 pad 1: Net-(J15-Pad1) -> Net-(F1-Pad2)
- J6 pad 1: /+5V1 -> +5V
- J6 pad 5: /+5V2 -> +5V
- SW4 pad : GND -> (no net)
- SW4 pad 1: Net-(J15-Pad1) -> Net-(F1-Pad1)
- SW4 pad 2: Net-(C31-Pad2) -> +5V
- U1 pad 1: HDMI_CLK+ -> HDMI_D0+
- U1 pad 3: HDMI_D0+ -> HDMI_CLK-
- U1 pad 4: HDMI_D0- -> HDMI_CLK+
- U1 pad 6: HDMI_CLK- -> HDMI_D0-
- U4 pad 10: CH376_1_CLK -> CH376_1_INT
- U4 pad 11: LED_Booted -> CH376_1_MOSI
- U4 pad 12: CH376_1_MOSI -> CH376_1_MISO
- U4 pad 13: LED_Eth -> CH376_2_CS
- U4 pad 14: CH376_1_MISO -> SW_4
- U4 pad 15: LED_Flash -> BTN_RST
- U4 pad 16: CH376_1_RST -> SW_3
- U4 pad 17: LED_USB0 -> CH376_2_RST
- U4 pad 18: CH376_1_INT -> SW_2
- U4 pad 19: LED_USB1 -> CH376_2_INT
- U4 pad 20: CH376_2_CS -> CH376_2_MOSI
- U4 pad 21: Net-(U4-Pad21) -> CH376_2_MISO
- U4 pad 23: CH376_2_MOSI -> LED_Booted
- U4 pad 24: CH376_2_MISO -> SW_1
- U4 pad 25: CH376_2_RST -> LED_USB0
- U4 pad 26: CH376_2_INT -> PS2_CLK
- U4 pad 27: Ext_GPIO_0 -> Net-(U4-Pad27)
- U4 pad 28: Ext_GPIO_1 -> PS2_Data
- U4 pad 29: Ext_GPIO_2 -> I2S_MCLK
- U4 pad 30: Ext_GPIO_3 -> Net-(U4-Pad30)
- U4 pad 31: Ext_GPIO_4 -> I2S_LRCLK
- U4 pad 32: Ext_GPIO_5 -> Ext_TX
- U4 pad 33: Ext_GPIO_6 -> I2S_SCLK
- U4 pad 34: Ext_GPIO_7 -> Ext_RX
- U4 pad 35: Net-(J8-Pad19) -> I2S_SDIN
- U4 pad 36: Ext_TX -> Net-(U4-Pad36)
- U4 pad 38: Ext_RX -> Net-(U4-Pad38)
- U4 pad 39: Net-(J8-Pad15) -> Flash_HOLD_IO3
- U4 pad 40: Ext_MISO -> Net-(U4-Pad40)
- U4 pad 41: Net-(J8-Pad13) -> Flash_MOSI_IO0
- U4 pad 42: Ext_MOSI -> Net-(U4-Pad42)
- U4 pad 43: Net-(J8-Pad11) -> Flash_CLK
- U4 pad 44: Ext_CLK -> Net-(U4-Pad44)
- U4 pad 45: Net-(J8-Pad9) -> Flash_MISO_IO1
- U4 pad 46: Ext_CS -> Net-(U4-Pad46)
- U4 pad 47: Net-(J8-Pad7) -> Flash_WP_IO2
- U4 pad 48: Ext_GP -> Net-(U4-Pad48)
- U4 pad 49: Net-(J8-Pad5) -> FPGC_TX
- U4 pad 50: W5500_MISO -> Flash_CS
- U4 pad 51: Net-(J8-Pad3) -> FPGC_RX
- U4 pad 52: W5500_RST -> Net-(U4-Pad52)
- U4 pad 53: Net-(J8-Pad1) -> FPGC_DTR
- U4 pad 54: W5500_INT -> Net-(U4-Pad54)
- U4 pad 55: FPGC_RX -> W5500_MISO
- U4 pad 56: W5500_CS -> W5500_RST
- U4 pad 57: FPGC_DTR -> W5500_INT
- U4 pad 58: W5500_CLK -> W5500_CS
- U4 pad 59: FPGC_TX -> W5500_CLK
- U4 pad 7: PS2_CLK -> CH376_1_CS
- U4 pad 8: CH376_1_CS -> CH376_1_CLK
- U4 pad 9: PS2_Data -> CH376_1_RST
- U5 pad 10: SW_1 -> LED_I2S
- U5 pad 11: Flash_MOSI_IO0 -> Ext_CLK
- U5 pad 12: BTN_RST -> LED_FSX
- U5 pad 13: Flash_HOLD_IO3 -> Ext_MOSI
- U5 pad 14: Flash_CLK -> LED_VideoOutput
- U5 pad 15: Flash_MISO_IO1 -> Ext_MISO
- U5 pad 16: Flash_WP_IO2 -> LED_Eth
- U5 pad 17: Flash_CS -> Ext_GPIO_7
- U5 pad 18: LED_I2S -> LED_SPImode
- U5 pad 19: DAC_D7 -> Ext_GPIO_6
- U5 pad 20: LED_FSX -> LED_Flash
- U5 pad 21: DAC_D6 -> Ext_GPIO_5
- U5 pad 22: LED_SPImode -> LED_USB1
- U5 pad 23: DAC_D5 -> Ext_GPIO_4
- U5 pad 24: LED_VideoOutput -> DAC_D0
- U5 pad 25: DAC_D4 -> Ext_GPIO_3
- U5 pad 26: LED_PS2 -> DAC_D1
- U5 pad 27: DAC_D3 -> Ext_GPIO_2
- U5 pad 28: I2S_MCLK -> DAC_D2
- U5 pad 29: DAC_D2 -> Ext_GPIO_1
- U5 pad 30: I2S_LRCLK -> DAC_D3
- U5 pad 31: DAC_D1 -> Ext_GPIO_0
- U5 pad 32: I2S_SCLK -> DAC_D4
- U5 pad 33: DAC_D0 -> Net-(U5-Pad33)
- U5 pad 34: I2S_SDIN -> DAC_D5
- U5 pad 36: Net-(J7-Pad1) -> DAC_D6
- U5 pad 38: Net-(J7-Pad3) -> DAC_D7
- U5 pad 45: HDMI_CLK- -> Net-(U5-Pad45)
- U5 pad 47: HDMI_CLK+ -> Net-(U5-Pad47)
- U5 pad 49: HDMI_D0- -> HDMI_D2+
- U5 pad 50: Net-(J7-Pad15) -> HDMI_D2-
- U5 pad 51: HDMI_D0+ -> HDMI_D1+
- U5 pad 52: Net-(J7-Pad17) -> HDMI_D1-
- U5 pad 53: HDMI_D1- -> HDMI_D0+
- U5 pad 54: Net-(J7-Pad19) -> HDMI_D0-
- U5 pad 55: HDMI_D1+ -> HDMI_CLK+
- U5 pad 56: Net-(U5-Pad56) -> HDMI_CLK-
- U5 pad 57: HDMI_D2- -> Net-(U5-Pad57)
- U5 pad 59: HDMI_D2+ -> Net-(U5-Pad59)
- U5 pad 7: SW_4 -> Ext_GP
- U5 pad 8: SW_3 -> LED_PS2
- U5 pad 9: SW_2 -> Ext_CS
- U6 pad 1: HDMI_D1- -> HDMI_D2+
- U6 pad 3: HDMI_D2- -> HDMI_D1-
- U6 pad 4: HDMI_D2+ -> HDMI_D1+
- U6 pad 6: HDMI_D1+ -> HDMI_D2-
Routing:
- net +5V: track 0.00 -> 336.5 mm, vias 0 -> 6
- net GND: track 0.00 -> 127.5 mm, vias 0 -> 46
- net Net-(J4-Pad1): track 0.00 -> 110.9 mm, vias 0 -> 3
- net +3V3: track 0.00 -> 104.5 mm, vias 0 -> 33
- net Net-(D12-Pad1): track 0.00 -> 88.2 mm
- net Audio_Mono: track 0.00 -> 87.1 mm, vias 0 -> 5
- net Net-(D11-Pad1): track 0.00 -> 87.1 mm
- net Net-(F1-Pad1): track 0.00 -> 75.7 mm, vias 0 -> 1
- net LED_USB1: track 0.00 -> 66.0 mm
- net LED_Flash: track 0.00 -> 61.3 mm
- net LED_SPImode: track 0.00 -> 56.6 mm
- net LED_Eth: track 0.00 -> 51.9 mm
- net LED_USB0: track 0.00 -> 50.7 mm, vias 0 -> 1
- net LED_Booted: track 0.00 -> 50.0 mm, vias 0 -> 1
- net /Ring1: track 0.00 -> 47.2 mm, vias 0 -> 2
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Other:
- board text removed: "LOGO"

Commit message: Basically finished the new PCB design
Parts:
- added C10: 47uF, Capacitor_SMD:C_0805_2012Metric_Pad1.18x1.45mm_HandSolder, B.Cu at (90.2, 58.4)
- added C11: 47uF, Capacitor_SMD:C_0805_2012Metric_Pad1.18x1.45mm_HandSolder, B.Cu at (90.2, 119.4)
- added C33: 47uF, Capacitor_SMD:C_0805_2012Metric_Pad1.18x1.45mm_HandSolder, B.Cu at (166.4, 119.4)
- added C34: 47uF, Capacitor_SMD:C_0805_2012Metric_Pad1.18x1.45mm_HandSolder, B.Cu at (103.1, 39.1)
- added C35: 47uF, Capacitor_SMD:C_0805_2012Metric_Pad1.18x1.45mm_HandSolder, B.Cu at (103.1, 36.8)
- added REF**: PinSocket_2x10_P2.54mm_Vertical, debugSocket:debugSocket2x10, F.Cu at (132.7, 102.9)
- added REF**: PinSocket_2x10_P2.54mm_Vertical, debugSocket:debugSocket2x10, F.Cu at (132.7, 97.8)
- C16: moved to B.Cu
- moved C17 1.56 mm to (103.1, 41.4), turned to 0 degrees
- moved LOGO 1.42 mm to (98.9, 49.9)
- moved C31 0.64 mm to (166.4, 127.0)
- moved C14 0.23 mm to (111.8, 87.4)
- renumbered IC1 to U10
Routing:
- net GND: track 127.5 -> 135.1 mm, vias 46 -> 45
- net Net-(J4-Pad1): track 110.9 -> 103.4 mm, vias 3 -> 0
- net +5V: track 336.5 -> 342.3 mm
- net (no net): track 0.00 -> 3.86 mm, vias 0 -> 2
- net +3V3: track 104.5 -> 107.7 mm, vias 33 -> 31
- net Audio_Mono: track 87.1 -> 84.0 mm, vias 5 -> 3
- net /Ring1: track 47.2 -> 45.0 mm
- net Ext_TX: vias 0 -> 2
- net Ext_RX: vias 0 -> 2
Other:
- board text added: "Config"
- board text added: "Design by: B4rt"
- board text added: "Ethernet"
- board text added: "FPGC I/O Board"
- board text added: "I2S"
- board text added: "OFF"
- board text added: "ON"
- board text added: "Power/ Data"
- board text added: "QSPI"
- board text added: "Reboot"
- board text added: "Reset"
- board text added: "SPI Flash"
- board text added: "USB"
- board text added: "USB Host"
- board text added: "USB/UART"
- board text added: "V3.0"
- board text added: "Video"
- board text added: "Video DAC"
- board text added: "nConfig"
- board text removed: "B4RT"
- board text removed: "Design by"
- board text removed: "SPI Mode"

Commit message: Added gerbers
Connections:
- SW4 pad 4: (no net) -> GND
Routing:
- net GND: track 135.1 -> 138.9 mm, vias 45 -> 47
- net (no net): track 3.86 -> 0.00 mm, vias 2 -> 0
